Commit message: anytrack v1 && simulation integration

File: ros/src/simulation/description/gazebo.xacro (robot description, xacro)
@@ -4,5 +4,8 @@
         <material>Gazebo/Green</material>
     </gazebo>
-    <joint name="camera_optical_joint" type="fixed">
+    <gazebo reference="cam1_link">
+        <material>Gazebo/Red</material>
+    </gazebo>
+    <joint name="cam0_optical_joint" type="fixed">
         <origin xyz="0 0 0" rpy="-1.571 0 -1.571" />
         <parent link="cam0_link" />
@@ -16,5 +19,4 @@
             <camera name="cam0">
                 <horizontal_fov>1.3962634</horizontal_fov>
-                <!-- <horizontal_fov>655.67987</horizontal_fov> -->
                 <image>
                     <width>1280</width>
@@ -27,6 +29,35 @@
                 </clip>
             </camera>
-            <plugin name="camera_controller" filename="libgazebo_ros_camera.so">
-                <frame_name>camera_link_optical</frame_name>
+            <plugin name="cam0_controller" filename="libgazebo_ros_camera.so">
+                <frame_name>cam0_link_optical</frame_name>
+                <min_depth>0.1</min_depth>
+                <max_depth>500</max_depth>
+            </plugin>
+        </sensor>
+    </gazebo>
+    <joint name="cam1_optical_joint" type="fixed">
+        <origin xyz="0 0 0" rpy="-1.571 0 -1.571" />
+        <parent link="cam1_link" />
+        <child link="cam1_link_optical" />
+    </joint>
+    <link name="cam1_link_optical"></link>
+    <gazebo reference="cam1_link">
+        <sensor type="camera" name="cam1">
+            <update_rate>30</update_rate>
+            <visualize>true</visualize>
+            <camera name="cam1">
+                <horizontal_fov>1.3962634</horizontal_fov>
+                <image>
+                    <width>1280</width>
+                    <height>720</height>
+                    <format>BGR8</format>
+                </image>
+                <clip>
+                    <near>0.02</near>
+                    <far>300</far>
+                </clip>
+            </camera>
+            <plugin name="cam1_controller" filename="libgazebo_ros_camera.so">
+                <frame_name>cam1_link_optical</frame_name>
                 <min_depth>0.1</min_depth>
                 <max_depth>500</max_depth>

File: ros/src/simulation/description/simulation.urdf.xacro (robot description, xacro)
@@ -31,6 +31,6 @@
         </xacro:inertial_box>
     </link>
-    <!-- <joint name="cam1_joint" type="fixed">
-        <origin xyz="2 1 1" rpy="1.3 0 0"/>
+    <joint name="cam1_joint" type="fixed">
+        <origin xyz="2 -2 1" rpy="0 0 ${pi/4}"/>
         <parent link="world"/>
         <child link="cam1_link"/>
@@ -58,9 +58,9 @@
             <origin xyz="0.0 0 0" rpy="0 0 0"/>
         </xacro:inertial_box>
-    </link> -->
+    </link>
     <!-- <gazebo reference="cam0_link">
         <material>Gazebo/Green</material>
-    </gazebo> -->
-    <!-- <gazebo reference="cam1_link">
+    </gazebo>
+    <gazebo reference="cam1_link">
         <material>Gazebo/Red</material>
     </gazebo> -->
