Commit message: simulation calibration working kinda

File: ros/src/simulation/description/simulation.urdf.xacro (robot description, xacro)
@@ -32,5 +32,6 @@
     </link>
     <joint name="cam1_joint" type="fixed">
-        <origin xyz="2 -2 1" rpy="0 0 ${pi/4}"/>
+        <!-- <origin xyz="2 -2 1" rpy="0 0 ${pi/4}"/> -->
+        <origin xyz="0 1 1" rpy="0 0 0"/>
         <parent link="world"/>
         <child link="cam1_link"/>

Commit message: live calibration working

File: ros/src/simulation/description/simulation.urdf.xacro (robot description, xacro)
@@ -60,68 +60,4 @@
         </xacro:inertial_box>
     </link>
-    <!-- <gazebo reference="cam0_link">
-        <material>Gazebo/Green</material>
-    </gazebo>
-    <gazebo reference="cam1_link">
-        <material>Gazebo/Red</material>
-    </gazebo> -->
-    <!-- <joint name="cam0_optical_joint" type="fixed">
-        <origin xyz="0 0 0" rpy="-1.571 0 -1.571" />
-        <parent link="cam0_link" />
-        <child link="cam0_link_optical" />
-    </joint>
-    <link name="cam0_link_optical"></link>
-    <gazebo reference="cam0_link">
-        <sensor type="camera" name="cam0">
-            <update_rate>30</update_rate>
-            <visualize>true</visualize>
-            <camera name="cam0">
-                <horizontal_fov>655.67987</horizontal_fov>
-                <image>
-                    <width>1280</width>
-                    <height>720</height>
-                    <format>R8B8G8</format>
-                </image>
-                <clip>
-                    <near>0.02</near>
-                    <far>300</far>
-                </clip>
-            </camera>
-            <plugin name="camera_controller" filename="libgazebo_ros_camera.so">
-                <frame_name>camera_link_optical</frame_name>
-                <min_depth>0.1</min_depth>
-                <max_depth>500</max_depth>
-            </plugin>
-        </sensor>
-    </gazebo> -->
-    <!-- <joint name="cam1_optical_joint" type="fixed">
-        <origin xyz="0 0 0" rpy="-1.571 0 -1.571" />
-        <parent link="cam1_link" />
-        <child link="cam1_link_optical" />
-    </joint>
-    <link name="cam1_link_optical"></link>
-    <gazebo reference="cam1_link">
-        <sensor type="camera" name="cam1">
-            <update_rate>30</update_rate>
-            <visualize>true</visualize>
-            <camera name="cam1">
-                <horizontal_fov>655.67987</horizontal_fov>
-                <image>
-                    <width>1280</width>
-                    <height>720</height>
-                    <format>R8B8G8</format>
-                </image>
-                <clip>
-                    <near>0.02</near>
-                    <far>300</far>
-                </clip>
-            </camera>
-            <plugin name="camera_controller" filename="libgazebo_ros_camera.so">
-                <frame_name>camera_link_optical</frame_name>
-                <min_depth>0.1</min_depth>
-                <max_depth>500</max_depth>
-            </plugin>
-        </sensor>
-    </gazebo> -->
     <xacro:include filename="gazebo.xacro" />
 </robot>
