Commit message: cleanup ros

File: ros/install/simulation/share/simulation/description/gazebo.xacro (robot description, xacro)
@@ -1 +1,67 @@
-/home/ALEX/anytrack/ros/src/simulation/description/gazebo.xacro
+<?xml version="1.0"?>
+<robot xmlns:xacro="http://www.ros.org/wiki/xacro">
+    <gazebo reference="cam0_link">
+        <material>Gazebo/Green</material>
+    </gazebo>
+    <gazebo reference="cam1_link">
+        <material>Gazebo/Red</material>
+    </gazebo>
+    <joint name="cam0_optical_joint" type="fixed">
+        <origin xyz="0 0 0" rpy="-1.571 0 -1.571" />
+        <parent link="cam0_link" />
+        <child link="cam0_link_optical" />
+    </joint>
+    <link name="cam0_link_optical"></link>
+    <gazebo reference="cam0_link">
+        <sensor type="camera" name="cam0">
+            <update_rate>30</update_rate>
+            <visualize>true</visualize>
+            <camera name="cam0">
+                <horizontal_fov>1.3962634</horizontal_fov>
+                <image>
+                    <width>1280</width>
+                    <height>720</height>
+                    <format>BGR8</format>
+                </image>
+                <clip>
+                    <near>0.02</near>
+                    <far>300</far>
+                </clip>
+            </camera>
+            <plugin name="cam0_controller" filename="libgazebo_ros_camera.so">
+                <frame_name>cam0_link_optical</frame_name>
+                <min_depth>0.1</min_depth>
+                <max_depth>500</max_depth>
+            </plugin>
+        </sensor>
+    </gazebo>
+    <joint name="cam1_optical_joint" type="fixed">
+        <origin xyz="0 0 0" rpy="-1.571 0 -1.571" />
+        <parent link="cam1_link" />
+        <child link="cam1_link_optical" />
+    </joint>
+    <link name="cam1_link_optical"></link>
+    <gazebo reference="cam1_link">
+        <sensor type="camera" name="cam1">
+            <update_rate>30</update_rate>
+            <visualize>true</visualize>
+            <camera name="cam1">
+                <horizontal_fov>1.3962634</horizontal_fov>
+                <image>
+                    <width>1280</width>
+                    <height>720</height>
+                    <format>BGR8</format>
+                </image>
+                <clip>
+                    <near>0.02</near>
+                    <far>300</far>
+                </clip>
+            </camera>
+            <plugin name="cam1_controller" filename="libgazebo_ros_camera.so">
+                <frame_name>cam1_link_optical</frame_name>
+                <min_depth>0.1</min_depth>
+                <max_depth>500</max_depth>
+            </plugin>
+        </sensor>
+    </gazebo>
+</robot>

File: ros/install/simulation/share/simulation/description/include.xacro (robot description, xacro)
@@ -1 +1,30 @@
-/home/ALEX/anytrack/ros/src/simulation/description/include.xacro
+<?xml version="1.0"?>
+<robot xmlns:xacro="http://www.ros.org/wiki/xacro" >
+    <xacro:macro name="inertial_sphere" params="mass radius *origin">
+        <inertial>
+            <xacro:insert_block name="origin"/>
+            <mass value="${mass}" />
+            <inertia ixx="${(2/5) * mass * (radius*radius)}" ixy="0.0" ixz="0.0"
+                    iyy="${(2/5) * mass * (radius*radius)}" iyz="0.0"
+                    izz="${(2/5) * mass * (radius*radius)}" />
+        </inertial>
+    </xacro:macro>
+    <xacro:macro name="inertial_box" params="mass x y z *origin">
+        <inertial>
+            <xacro:insert_block name="origin"/>
+            <mass value="${mass}" />
+            <inertia ixx="${(1/12) * mass * (y*y+z*z)}" ixy="0.0" ixz="0.0"
+                    iyy="${(1/12) * mass * (x*x+z*z)}" iyz="0.0"
+                    izz="${(1/12) * mass * (x*x+y*y)}" />
+        </inertial>
+    </xacro:macro>
+    <xacro:macro name="inertial_cylinder" params="mass length radius *origin">
+        <inertial>
+            <xacro:insert_block name="origin"/>
+            <mass value="${mass}" />
+            <inertia ixx="${(1/12) * mass * (3*radius*radius + length*length)}" ixy="0.0" ixz="0.0"
+                    iyy="${(1/12) * mass * (3*radius*radius + length*length)}" iyz="0.0"
+                    izz="${(1/2) * mass * (radius*radius)}" />
+        </inertial>
+    </xacro:macro>
+</robot>

File: ros/install/simulation/share/simulation/description/simulation.urdf.xacro (robot description, xacro)
@@ -1 +1,63 @@
-/home/ALEX/anytrack/ros/src/simulation/description/simulation.urdf.xacro
+<?xml version="1.0"?>
+<robot xmlns:xacro="http://www.ros.org/wiki/xacro"  name="robot">
+    <xacro:include filename="include.xacro" />
+    <link name="world"></link>
+    <joint name="cam0_joint" type="fixed">
+        <origin xyz="0 0 1" rpy="0 0 0"/>
+        <parent link="world"/>
+        <child link="cam0_link"/>
+    </joint>
+    <link name="cam0_link">
+        <visual>
+            <origin xyz="-0.03 0 0" rpy="0 0 0"/>
+            <geometry>
+                <box size="0.06 0.15 0.15" />
+            </geometry>
+        </visual>
+        <visual>
+            <origin xyz="0.03 0 0" rpy="0 ${pi/2} 0"/>
+            <geometry>
+                <cylinder length="0.06" radius="0.04" />
+            </geometry>
+        </visual>
+        <collision>
+            <origin xyz="0.0 0 0" rpy="0 0 0"/>
+            <geometry>
+                <box size="0.12 0.15 0.15" />
+            </geometry>
+        </collision>
+        <xacro:inertial_box mass="0.1" x="0.12" y="0.15" z="0.15">
+            <origin xyz="0.0 0 0" rpy="0 0 0"/>
+        </xacro:inertial_box>
+    </link>
+    <joint name="cam1_joint" type="fixed">
+        <!-- <origin xyz="2 -2 1" rpy="0 0 ${pi/4}"/> -->
+        <origin xyz="0 1 1" rpy="0 0 0"/>
+        <parent link="world"/>
+        <child link="cam1_link"/>
+    </joint>
+    <link name="cam1_link">
+        <visual>
+            <origin xyz="-0.03 0 0" rpy="0 0 0"/>
+            <geometry>
+                <box size="0.06 0.15 0.15" />
+            </geometry>
+        </visual>
+        <visual>
+            <origin xyz="0.03 0 0" rpy="0 ${pi/2} 0"/>
+            <geometry>
+                <cylinder length="0.06" radius="0.04" />
+            </geometry>
+        </visual>
+        <collision>
+            <origin xyz="0.0 0 0" rpy="0 0 0"/>
+            <geometry>
+                <box size="0.12 0.15 0.15" />
+            </geometry>
+        </collision>
+        <xacro:inertial_box mass="0.1" x="0.12" y="0.15" z="0.15">
+            <origin xyz="0.0 0 0" rpy="0 0 0"/>
+        </xacro:inertial_box>
+    </link>
+    <xacro:include filename="gazebo.xacro" />
+</robot>

Commit message: new calibration algorithm with feedback

File: ros/install/simulation/share/simulation/description/gazebo.xacro (robot description, xacro)
@@ -1,67 +1 @@
-<?xml version="1.0"?>
-<robot xmlns:xacro="http://www.ros.org/wiki/xacro">
-    <gazebo reference="cam0_link">
-        <material>Gazebo/Green</material>
-    </gazebo>
-    <gazebo reference="cam1_link">
-        <material>Gazebo/Red</material>
-    </gazebo>
-    <joint name="cam0_optical_joint" type="fixed">
-        <origin xyz="0 0 0" rpy="-1.571 0 -1.571" />
-        <parent link="cam0_link" />
-        <child link="cam0_link_optical" />
-    </joint>
-    <link name="cam0_link_optical"></link>
-    <gazebo reference="cam0_link">
-        <sensor type="camera" name="cam0">
-            <update_rate>30</update_rate>
-            <visualize>true</visualize>
-            <camera name="cam0">
-                <horizontal_fov>1.3962634</horizontal_fov>
-                <image>
-                    <width>1280</width>
-                    <height>720</height>
-                    <format>BGR8</format>
-                </image>
-                <clip>
-                    <near>0.02</near>
-                    <far>300</far>
-                </clip>
-            </camera>
-            <plugin name="cam0_controller" filename="libgazebo_ros_camera.so">
-                <frame_name>cam0_link_optical</frame_name>
-                <min_depth>0.1</min_depth>
-                <max_depth>500</max_depth>
-            </plugin>
-        </sensor>
-    </gazebo>
-    <joint name="cam1_optical_joint" type="fixed">
-        <origin xyz="0 0 0" rpy="-1.571 0 -1.571" />
-        <parent link="cam1_link" />
-        <child link="cam1_link_optical" />
-    </joint>
-    <link name="cam1_link_optical"></link>
-    <gazebo reference="cam1_link">
-        <sensor type="camera" name="cam1">
-            <update_rate>30</update_rate>
-            <visualize>true</visualize>
-            <camera name="cam1">
-                <horizontal_fov>1.3962634</horizontal_fov>
-                <image>
-                    <width>1280</width>
-                    <height>720</height>
-                    <format>BGR8</format>
-                </image>
-                <clip>
-                    <near>0.02</near>
-                    <far>300</far>
-                </clip>
-            </camera>
-            <plugin name="cam1_controller" filename="libgazebo_ros_camera.so">
-                <frame_name>cam1_link_optical</frame_name>
-                <min_depth>0.1</min_depth>
-                <max_depth>500</max_depth>
-            </plugin>
-        </sensor>
-    </gazebo>
-</robot>
+/home/ALEX/anytrack/ros/src/simulation/description/gazebo.xacro

File: ros/install/simulation/share/simulation/description/include.xacro (robot description, xacro)
@@ -1,30 +1 @@
-<?xml version="1.0"?>
-<robot xmlns:xacro="http://www.ros.org/wiki/xacro" >
-    <xacro:macro name="inertial_sphere" params="mass radius *origin">
-        <inertial>
-            <xacro:insert_block name="origin"/>
-            <mass value="${mass}" />
-            <inertia ixx="${(2/5) * mass * (radius*radius)}" ixy="0.0" ixz="0.0"
-                    iyy="${(2/5) * mass * (radius*radius)}" iyz="0.0"
-                    izz="${(2/5) * mass * (radius*radius)}" />
-        </inertial>
-    </xacro:macro>
-    <xacro:macro name="inertial_box" params="mass x y z *origin">
-        <inertial>
-            <xacro:insert_block name="origin"/>
-            <mass value="${mass}" />
-            <inertia ixx="${(1/12) * mass * (y*y+z*z)}" ixy="0.0" ixz="0.0"
-                    iyy="${(1/12) * mass * (x*x+z*z)}" iyz="0.0"
-                    izz="${(1/12) * mass * (x*x+y*y)}" />
-        </inertial>
-    </xacro:macro>
-    <xacro:macro name="inertial_cylinder" params="mass length radius *origin">
-        <inertial>
-            <xacro:insert_block name="origin"/>
-            <mass value="${mass}" />
-            <inertia ixx="${(1/12) * mass * (3*radius*radius + length*length)}" ixy="0.0" ixz="0.0"
-                    iyy="${(1/12) * mass * (3*radius*radius + length*length)}" iyz="0.0"
-                    izz="${(1/2) * mass * (radius*radius)}" />
-        </inertial>
-    </xacro:macro>
-</robot>
+/home/ALEX/anytrack/ros/src/simulation/description/include.xacro

File: ros/install/simulation/share/simulation/description/simulation.urdf.xacro (robot description, xacro)
@@ -1,63 +1 @@
-<?xml version="1.0"?>
-<robot xmlns:xacro="http://www.ros.org/wiki/xacro"  name="robot">
-    <xacro:include filename="include.xacro" />
-    <link name="world"></link>
-    <joint name="cam0_joint" type="fixed">
-        <origin xyz="0 0 1" rpy="0 0 0"/>
-        <parent link="world"/>
-        <child link="cam0_link"/>
-    </joint>
-    <link name="cam0_link">
-        <visual>
-            <origin xyz="-0.03 0 0" rpy="0 0 0"/>
-            <geometry>
-                <box size="0.06 0.15 0.15" />
-            </geometry>
-        </visual>
-        <visual>
-            <origin xyz="0.03 0 0" rpy="0 ${pi/2} 0"/>
-            <geometry>
-                <cylinder length="0.06" radius="0.04" />
-            </geometry>
-        </visual>
-        <collision>
-            <origin xyz="0.0 0 0" rpy="0 0 0"/>
-            <geometry>
-                <box size="0.12 0.15 0.15" />
-            </geometry>
-        </collision>
-        <xacro:inertial_box mass="0.1" x="0.12" y="0.15" z="0.15">
-            <origin xyz="0.0 0 0" rpy="0 0 0"/>
-        </xacro:inertial_box>
-    </link>
-    <joint name="cam1_joint" type="fixed">
-        <!-- <origin xyz="2 -2 1" rpy="0 0 ${pi/4}"/> -->
-        <origin xyz="0 1 1" rpy="0 0 0"/>
-        <parent link="world"/>
-        <child link="cam1_link"/>
-    </joint>
-    <link name="cam1_link">
-        <visual>
-            <origin xyz="-0.03 0 0" rpy="0 0 0"/>
-            <geometry>
-                <box size="0.06 0.15 0.15" />
-            </geometry>
-        </visual>
-        <visual>
-            <origin xyz="0.03 0 0" rpy="0 ${pi/2} 0"/>
-            <geometry>
-                <cylinder length="0.06" radius="0.04" />
-            </geometry>
-        </visual>
-        <collision>
-            <origin xyz="0.0 0 0" rpy="0 0 0"/>
-            <geometry>
-                <box size="0.12 0.15 0.15" />
-            </geometry>
-        </collision>
-        <xacro:inertial_box mass="0.1" x="0.12" y="0.15" z="0.15">
-            <origin xyz="0.0 0 0" rpy="0 0 0"/>
-        </xacro:inertial_box>
-    </link>
-    <xacro:include filename="gazebo.xacro" />
-</robot>
+/home/ALEX/anytrack/ros/src/simulation/description/simulation.urdf.xacro
